File: pcb/SSR.kicad_pcb (KiCad board)
At the start: 2 copper layers, 53 x 36.9 mm, 20 parts, among them J1 Conn_01x04, J2 IN_AC, J3 RESISTENCIA, U1 MOC3021M, U3 4N25

Commit message: Añadido Zener
Parts:
- removed kibuzzard-635BB698: G***, kibuzzard-635BB698
- removed kibuzzard-635BB6A0: G***, kibuzzard-635BB6A0
- removed kibuzzard-635EA6AB: G***, kibuzzard-635EA6AB
- added D4: MMSZ4684-TP, Diode_SMD:D_SOD-123, F.Cu at (173.8, 106.6)
- R1: value 270 -> 1K
- R2: value 330 -> 220
- moved D2 5.17 mm to (179.9, 107.0)
- moved R9 2.13 mm to (144.7, 99.4)
- moved R1 1.39 mm to (144.7, 85.2), turned to 90 degrees
- moved R2 0.37 mm to (144.7, 92.3)
- moved LD1 0.19 mm to (140.9, 83.5)
Routing:
- net Net-(LD1-A): track 14.1 -> 3.30 mm
- net Net-(D2--): track 31.1 -> 41.1 mm
- net Net-(D2-+): track 22.6 -> 31.8 mm
- net Net-(D2-Pad4): track 28.7 -> 33.1 mm
- net ZC: track 14.7 -> 18.3 mm
- net /NEUTRO: track 27.9 -> 25.3 mm
- net +5V: track 11.2 -> 12.8 mm
- net /PWM: track 14.6 -> 13.7 mm
Other:
- board text added: "AC-IN"
- board text added: "LOAD"
- board text added: "ON"
